File: KiCad/reddit/reddit.kicad_pcb (KiCad board)
At the start: 2 copper layers, 52.6 x 93.1 mm, 6 parts

Commit message: version 1.2
Parts:
- added G***: LOGO, reddit:DEFCON_silkscreen_mod, F.Cu at (149.6, 116.6)
- added G***: LOGO, reddit:reddit_logo_silkscreen, B.Cu at (121.8, 63.0)
- added REF**: MountingHole_3.2mm_M3_ISO14580, MountingHole:MountingHole_3.2mm_M3_ISO14580, F.Cu at (135.1, 59.2)
Routing:
- net (no net): vias 1 -> 0

Commit message: version 1.3
Routing:
- net (no net): track 0.00 -> 313.8 mm, vias 0 -> 46

Commit message: version 1.3
Routing:
- net (no net): track 313.8 -> 422.3 mm, vias 46 -> 62
- net Net-(BT1-Pad2): track 64.8 -> 83.4 mm, vias 0 -> 4

Commit message: version 1.4
Routing:
- net Net-(BT1-Pad2): track 83.4 -> 80.1 mm, vias 4 -> 6
Other:
- board text added: "r/Defcon"
Changed lines of the file:
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@@
   (general
     (thickness 1.6)
-    (drawings 449)
-    (tracks 222)
+    (drawings 450)
+    (tracks 227)
     (zones 0)
     (modules 9)
@@
     )
   )
+  (gr_text r/Defcon (at 149.86 123.19) (layer F.SilkS)
+    (effects (font (size 1 1) (thickness 0.15)))
+  )
   (gr_line (start 149.606 111.4044) (end 151.892 105.2322) (layer F.SilkS) (width 0.3))
   (gr_line (start 139.1158 106.0704) (end 149.5806 111.4552) (layer F.SilkS) (width 0.3))
@@
   (segment (start 148.59 125.73) (end 149.86 125.73) (width 0.25) (layer F.Cu) (net 0))
   (segment (start 149.86 125.73) (end 154.94 120.65) (width 0.25) (layer F.Cu) (net 0))
+  (via (at 144.78 125.73) (size 0.8) (drill 0.4) (layers F.Cu B.Cu) (net 1))
+  (via (at 146.05 124.46) (size 0.8) (drill 0.4) (layers F.Cu B.Cu) (net 1))
   (via (at 148.59 124.46) (size 0.8) (drill 0.4) (layers F.Cu B.Cu) (net 1))
-  (via (at 144.78 124.46) (size 0.8) (drill 0.4) (layers F.Cu B.Cu) (net 1))
-  (via (at 149.86 123.19) (size 0.8) (drill 0.4) (layers F.Cu B.Cu) (net 1))
-  (via (at 143.51 124.46) (size 0.8) (drill 0.4) (layers F.Cu B.Cu) (net 1))
+  (via (at 143.51 125.73) (size 0.8) (drill 0.4) (layers F.Cu B.Cu) (net 1))
+  (via (at 146.05 121.92) (size 0.8) (drill 0.4) (layers F.Cu B.Cu) (net 1))
+  (via (at 142.24 125.73) (size 0.8) (drill 0.4) (layers F.Cu B.Cu) (net 1))
   (segment (start 138.43 110.49) (end 144.78 116.84) (width 0.25) (layer B.Cu) (net 1))
   (segment (start 144.78 116.84) (end 144.78 115.9256) (width 0.25) (layer B.Cu) (net 1))
@@
   (segment (start 139.192 83.8708) (end 158.4424 83.8708) (width 0.25) (layer B.Cu) (net 1))
   (segment (start 137.6172 85.4456) (end 139.192 83.8708) (width 0.25) (layer B.Cu) (net 1))
-  (segment (start 143.51 124.46) (end 143.51 120.65) (width 0.25) (layer F.Cu) (net 1))
-  (segment (start 143.51 120.65) (end 144.78 120.65) (width 0.25) (layer F.Cu) (net 1))
-  (segment (start 144.78 120.65) (end 147.32 123.19) (width 0.25) (layer F.Cu) (net 1))
-  (segment (start 147.32 123.19) (end 149.86 123.19) (width 0.25) (layer F.Cu) (net 1))
-  (segment (start 144.78 124.46) (end 144.78 121.92) (width 0.25) (layer F.Cu) (net 1))
-  (segment (start 144.78 121.92) (end 147.32 124.46) (width 0.25) (layer F.Cu) (net 1))
   (segment (start 147.32 124.46) (end 148.59 124.46) (width 0.25) (layer F.Cu) (net 1))
+  (segment (start 144.78 124.46) (end 143.51 125.73) (width 0.25) (layer F.Cu) (net 1))
+  (segment (start 147.32 124.46) (end 146.05 123.19) (width 0.25) (layer F.Cu) (net 1))
+  (segment (start 146.05 123.19) (end 144.78 123.19) (width 0.25) (layer F.Cu) (net 1))
+  (segment (start 144.78 123.19) (end 144.78 124.46) (width 0.25) (layer F.Cu) (net 1))
+  (segment (start 144.78 125.73) (end 146.05 124.46) (width 0.25) (layer F.Cu) (net 1))
+  (segment (start 142.24 125.73) (end 143.51 124.46) (width 0.25) (layer F.Cu) (net 1))
+  (segment (start 143.51 124.46) (end 143.51 123.19) (width 0.25) (layer F.Cu) (net 1))
+  (segment (start 143.51 123.19) (end 144.78 121.92) (width 0.25) (layer F.Cu) (net 1))
+  (segment (start 144.78 121.92) (end 146.05 121.92) (width 0.25) (layer F.Cu) (net 1))
   (segment (start 144.78 104.04) (end 144.0958 104.04) (width 0.25) (layer B.Cu) (net 2))
   (segment (start 140.4874 100.4316) (end 140.4874 94.1578) (width 0.25) (layer B.Cu) (net 2))
