File: KiCad/reddit/reddit.kicad_pcb (KiCad board)
At the start: 2 copper layers, 52.6 x 93.1 mm, 9 parts

Commit message: version 1.5
Parts:
- removed the G*** at (149.6, 116.6)
- added G***: LOGO, reddit:reddit_logo_silkscreen, F.Cu at (149.9, 116.8)
Routing:
- net (no net): track 422.3 -> 424.8 mm
- net Net-(BT1-Pad2): track 80.1 -> 77.8 mm
Other:
- board text added: "2023"
