File: KiCad/reddit/reddit.kicad_pcb (KiCad board)
At the start: 2 copper layers, 1 part

Commit message: schematic and components
Parts:
- added BT1: Battery_Cell, Battery:BatteryHolder_Keystone_3002_1x2032, B.Cu at (144.8, 116.8)
- added D1: LED, LED_SMD:LED_PLCC-2, B.Cu at (160.0, 83.8)
- added D2: LED, LED_SMD:LED_PLCC-2, B.Cu at (139.9, 86.4)
- added R1: R, Resistor_SMD:R_0805_2012Metric_Pad1.20x1.40mm_HandSolder, B.Cu at (141.0, 93.7)
Routing:
- net Net-(BT1-Pad2): track 0.00 -> 55.7 mm
- net Net-(D1-Pad2): track 0.00 -> 29.0 mm
- net Net-(BT1-Pad1): track 0.00 -> 10.9 mm

Commit message: revision 1.0
Parts:
- moved D2 0.81 mm to (139.1, 86.3)
- moved R1 0.73 mm to (140.5, 93.2)
- moved D1 0.09 mm to (159.9, 83.9)
- moved G*** 0.06 mm to (143.5, 100.3)
Routing:
- net Net-(BT1-Pad2): track 55.7 -> 64.8 mm
- net Net-(BT1-Pad1): track 10.9 -> 12.1 mm
- net Net-(D1-Pad2): track 29.0 -> 28.4 mm
- net (no net): vias 0 -> 1
Other:
- board outline added: 52.6 x 93.1 mm
- board text added: "TheDevilsVoice Y3t1 p0lr"

Commit message: version 1.1
Parts:
- added G***: LOGO, reddit:D3AD10C5_silkscreen, B.Cu at (150.3, 83.1)
Other:
- outline, holes or cut-outs redrawn

Commit message: testing
Other:
- net class Default removed
- board text added: "0.2000 mm / 0.0000 mm"
- board text added: "0.3000 mm"
- board text added: "1.6000 mm"
- board text added: "2"
- board text added: "52.6288 mm x 93.0910 mm"
- board text added: "BOARD CHARACTERISTICS"
- board text added: "Board Thickness:"
- board text added: "Board overall dimensions:"
- board text added: "Castellated pads:"
- board text added: "Copper Finish:"
- board text added: "Copper Layer Count:"
- board text added: "Edge card connectors:"
- board text added: "Impedance Control:"
- board text added: "Min hole diameter:"
- board text added: "Min track/spacing:"
- board text added: "No"
- board text added: "None"
- board text added: "Plated Board Edge:"
