File: kicad/reddit.kicad_sch (KiCad schematic)
At the start: 4 parts

Commit message: P0lr1 (#11)
* version 1.2

* version 1.3

* version 1.3

* version 1.4

* version 1.41

* version 1.5

* Upgrading to KiCad 6

* udpate the board files

* remove old files

Co-authored-by: franklin <2730246+devsecfranklin@users.noreply.github.com>
Parts:
- BT1: value (none) -> Battery_Cell; footprint (none) -> Battery:BatteryHolder_Keystone_3002_1x2032
- D1, D2: value (none) -> LED; footprint (none) -> LED_SMD:LED_PLCC-2
- R1: value (none) -> R; footprint (none) -> Resistor_SMD:R_0805_2012Metric_Pad1.20x1.40mm_HandSolder
Other:
- title: Shitty Add-On of Reddit avatar for DEFCON 2023 -> r/DEFCON
Changed lines of the file:
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@@
   (paper "A4")
   (title_block
-    (title "Shitty Add-On of Reddit avatar for DEFCON 2023")
-    (date "2022-08-23")
-    (rev "1.1")
+    (title "r/DEFCON")
+    (date "2022-08-25")
+    (rev "v1.5")
     (company "DE:AD:10:C5")
   )
@@
   (junction (at 128.27 95.25) (diameter 0) (color 0 0 0 0)
   )
-  (wire (pts (xy 88.9 78.74) (xy 88.9 85.09))
+  (wire (pts (xy 88.9 99.06) (xy 88.9 92.71))
+    (stroke (width 0) (type default) (color 0 0 0 0))
+  )
+  (wire (pts (xy 102.87 78.74) (xy 88.9 78.74))
+    (stroke (width 0) (type default) (color 0 0 0 0))
+  )
+  (wire (pts (xy 120.65 83.82) (xy 120.65 95.25))
     (stroke (width 0) (type default) (color 0 0 0 0))
   )
@@
     (stroke (width 0) (type default) (color 0 0 0 0))
   )
-  (wire (pts (xy 110.49 78.74) (xy 120.65 78.74))
-    (stroke (width 0) (type default) (color 0 0 0 0))
-  )
-  (wire (pts (xy 102.87 78.74) (xy 88.9 78.74))
+  (wire (pts (xy 88.9 78.74) (xy 88.9 85.09))
     (stroke (width 0) (type default) (color 0 0 0 0))
   )
@@
     (stroke (width 0) (type default) (color 0 0 0 0))
   )
+  (wire (pts (xy 128.27 99.06) (xy 88.9 99.06))
+    (stroke (width 0) (type default) (color 0 0 0 0))
+  )
   (wire (pts (xy 128.27 83.82) (xy 128.27 95.25))
     (stroke (width 0) (type default) (color 0 0 0 0))
   )
-  (wire (pts (xy 120.65 83.82) (xy 120.65 95.25))
-    (stroke (width 0) (type default) (color 0 0 0 0))
-  )
-  (wire (pts (xy 128.27 99.06) (xy 88.9 99.06))
-    (stroke (width 0) (type default) (color 0 0 0 0))
-  )
-  (wire (pts (xy 88.9 99.06) (xy 88.9 92.71))
+  (wire (pts (xy 110.49 78.74) (xy 120.65 78.74))
     (stroke (width 0) (type default) (color 0 0 0 0))
   )
@@
       (effects (font (size 1.27 1.27)) (justify left))
     )
-    (property "Value" "" (id 1) (at 91.8972 90.043 0)
+    (property "Value" "Battery_Cell" (id 1) (at 91.8972 90.043 0)
       (effects (font (size 1.27 1.27)) (justify left))
     )
-    (property "Footprint" "" (id 2) (at 88.9 88.646 90)
+    (property "Footprint" "Battery:BatteryHolder_Keystone_3002_1x2032" (id 2) (at 88.9 88.646 90)
       (effects (font (size 1.27 1.27)) hide)
     )
@@
     (in_bom yes) (on_board yes)
     (property "Reference" "R1" (id 0) (at 106.68 73.4822 90))
-    (property "Value" "" (id 1) (at 106.68 75.7936 90))
-    (property "Footprint" "" (id 2) (at 106.68 80.518 90)
+    (property "Value" "R" (id 1) (at 106.68 75.7936 90))
+    (property "Footprint" "Resistor_SMD:R_0805_2012Metric_Pad1.20x1.40mm_HandSolder" (id 2) (at 106.68 80.518 90)
       (effects (font (size 1.27 1.27)) hide)
     )
@@
     (in_bom yes) (on_board yes)
     (property "Reference" "D1" (id 0) (at 124.6378 77.343 0))
-    (property "Value" "" (id 1) (at 124.6378 79.6544 0))
-    (property "Footprint" "" (id 2) (at 124.46 83.82 0)
+    (property "Value" "LED" (id 1) (at 124.6378 79.6544 0))
+    (property "Footprint" "LED_SMD:LED_PLCC-2" (id 2) (at 124.46 83.82 0)
       (effects (font (size 1.27 1.27)) hide)
     )
@@
     (in_bom yes) (on_board yes)
     (property "Reference" "D2" (id 0) (at 124.6378 88.773 0))
-    (property "Value" "" (id 1) (at 124.6378 91.0844 0))
-    (property "Footprint" "" (id 2) (at 124.46 95.25 0)
+    (property "Value" "LED" (id 1) (at 124.6378 91.0844 0))
+    (property "Footprint" "LED_SMD:LED_PLCC-2" (id 2) (at 124.46 95.25 0)
       (effects (font (size 1.27 1.27)) hide)
     )
