File: pcb/reddit.kicad_sch (KiCad schematic)
At the start: 4 parts

Commit message: updates from p0lr
Parts:
- D1, D2: footprint LED_SMD:LED_PLCC-2 -> reddit:LED_PLCC-2_Reverse-Mount
Other:
- company: DE:AD:10:C5 -> (none)
- title: r/DEFCON -> (none)
Changed lines of the file:
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@@
 (kicad_sch (version 20211123) (generator eeschema)
   (paper "A4")
-  (title_block
-    (title "r/DEFCON")
-    (date "2022-08-25")
-    (rev "v1.5")
-    (company "DE:AD:10:C5")
+  (junction (at 128.27 95.25) (diameter 0) (color 0 0 0 0)
   )
   (junction (at 120.65 83.82) (diameter 0) (color 0 0 0 0)
   )
-  (junction (at 128.27 95.25) (diameter 0) (color 0 0 0 0)
-  )
-  (wire (pts (xy 88.9 99.06) (xy 88.9 92.71))
+  (wire (pts (xy 128.27 83.82) (xy 128.27 95.25))
     (stroke (width 0) (type default) (color 0 0 0 0))
   )
-  (wire (pts (xy 102.87 78.74) (xy 88.9 78.74))
+  (wire (pts (xy 110.49 78.74) (xy 120.65 78.74))
     (stroke (width 0) (type default) (color 0 0 0 0))
   )
-  (wire (pts (xy 120.65 83.82) (xy 120.65 95.25))
-    (stroke (width 0) (type default) (color 0 0 0 0))
-  )
-  (wire (pts (xy 120.65 78.74) (xy 120.65 83.82))
+  (wire (pts (xy 128.27 99.06) (xy 88.9 99.06))
     (stroke (width 0) (type default) (color 0 0 0 0))
   )
@@
     (stroke (width 0) (type default) (color 0 0 0 0))
   )
-  (wire (pts (xy 128.27 99.06) (xy 88.9 99.06))
+  (wire (pts (xy 102.87 78.74) (xy 88.9 78.74))
     (stroke (width 0) (type default) (color 0 0 0 0))
   )
-  (wire (pts (xy 128.27 83.82) (xy 128.27 95.25))
+  (wire (pts (xy 88.9 99.06) (xy 88.9 92.71))
     (stroke (width 0) (type default) (color 0 0 0 0))
   )
-  (wire (pts (xy 110.49 78.74) (xy 120.65 78.74))
+  (wire (pts (xy 120.65 83.82) (xy 120.65 95.25))
+    (stroke (width 0) (type default) (color 0 0 0 0))
+  )
+  (wire (pts (xy 120.65 78.74) (xy 120.65 83.82))
     (stroke (width 0) (type default) (color 0 0 0 0))
   )
@@
     (property "Reference" "D1" (id 0) (at 124.6378 77.343 0))
     (property "Value" "LED" (id 1) (at 124.6378 79.6544 0))
-    (property "Footprint" "LED_SMD:LED_PLCC-2" (id 2) (at 124.46 83.82 0)
+    (property "Footprint" "reddit:LED_PLCC-2_Reverse-Mount" (id 2) (at 124.46 83.82 0)
       (effects (font (size 1.27 1.27)) hide)
     )
@@
     (property "Reference" "D2" (id 0) (at 124.6378 88.773 0))
     (property "Value" "LED" (id 1) (at 124.6378 91.0844 0))
-    (property "Footprint" "LED_SMD:LED_PLCC-2" (id 2) (at 124.46 95.25 0)
+    (property "Footprint" "reddit:LED_PLCC-2_Reverse-Mount" (id 2) (at 124.46 95.25 0)
       (effects (font (size 1.27 1.27)) hide)
     )
@@
     )
     (path "/00000000-0000-0000-0000-000063003fc9"
-      (reference "D1") (unit 1) (value "LED") (footprint "LED_SMD:LED_PLCC-2")
+      (reference "D1") (unit 1) (value "LED") (footprint "reddit:LED_PLCC-2_Reverse-Mount")
     )
     (path "/00000000-0000-0000-0000-000063004530"
-      (reference "D2") (unit 1) (value "LED") (footprint "LED_SMD:LED_PLCC-2")
+      (reference "D2") (unit 1) (value "LED") (footprint "reddit:LED_PLCC-2_Reverse-Mount")
     )
     (path "/00000000-0000-0000-0000-000063003633"
